File: Drone.kicad_pcb (KiCad board)
At the start: 2 copper layers, 51 parts, among them J1 USB_C_Receptacle_USB2.0_16P, J2 Conn_01x02_Pin, J3 Conn_01x06_Socket, J4 Conn_01x06_Socket, Q1 AO3401A, Q2 2N7002, Q3 2N7002, Q4 2N7002, Q5 2N7002, U1 TP4056-42-ESOP8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

Commit message: V1 of PCB
Parts:
- removed C10: C, Capacitor_SMD:C_0603_1608Metric
- added C14: 1uf, Capacitor_SMD:C_0603_1608Metric, F.Cu at (134.5, 44.4)
- added C15: 1uf, Capacitor_SMD:C_0603_1608Metric, F.Cu at (84.3, 42.5)
- added C16: 1uf, Capacitor_SMD:C_0603_1608Metric, F.Cu at (89.0, 89.7)
- added C17: 1uf, Capacitor_SMD:C_0603_1608Metric, F.Cu at (133.0, 90.8)
- added D10: LED 5, LED_SMD:LED_0603_1608Metric, F.Cu at (94.8, 55.5)
- added D11: LED 6, LED_SMD:LED_0603_1608Metric, F.Cu at (103.4, 54.0)
- added D9: LED 4, LED_SMD:LED_0603_1608Metric, B.Cu at (98.3, 45.4)
- added J5: Conn_01x02_Socket, Connector_PinHeader_2.54mm:PinHeader_1x02_P2.54mm_Vertical, F.Cu at (136.3, 39.1)
- added J6: Conn_01x02_Socket, Connector_PinHeader_2.54mm:PinHeader_1x02_P2.54mm_Vertical, F.Cu at (81.2, 35.7)
- added J7: Conn_01x02_Socket, Connector_PinHeader_2.54mm:PinHeader_1x02_P2.54mm_Vertical, F.Cu at (82.0, 93.7)
- added J8: Conn_01x02_Socket, Connector_PinHeader_2.54mm:PinHeader_1x02_P2.54mm_Vertical, F.Cu at (138.2, 92.5)
- added R16: 10k, Resistor_SMD:R_0603_1608Metric, F.Cu at (126.9, 48.3)
- added R17: 10k, Resistor_SMD:R_0603_1608Metric, F.Cu at (92.2, 46.2)
- added R18: 10k, Resistor_SMD:R_0603_1608Metric, F.Cu at (93.0, 82.8)
- added R19: 10k, Resistor_SMD:R_0603_1608Metric, F.Cu at (129.5, 83.7)
- added R20: 1k, Resistor_SMD:R_0603_1608Metric, B.Cu at (98.3, 43.9)
- added R21: 1k, Resistor_SMD:R_0603_1608Metric, F.Cu at (90.4, 55.1)
- added R22: 1k, Resistor_SMD:R_0603_1608Metric, F.Cu at (105.0, 52.5)
- added SW1: SW_DPDT_x2, Button_Switch_THT:SW_PUSH_6mm, F.Cu at (126.2, 76.2)
- added SW2: RST, Button_Switch_THT:SW_PUSH_6mm, F.Cu at (104.3, 75.8)
- added SW3: BOOT, Button_Switch_THT:SW_PUSH_6mm, F.Cu at (97.8, 63.9)
- C6, C7, C9, R10, R11, R9, U3, U4, U5: moved to B.Cu
- J2: footprint Connector_PinHeader_2.54mm:PinHeader_1x06_P2.54mm_Vertical -> Connector_PinHeader_2.54mm:PinHeader_1x02_P2.54mm_Vertical
- J3, J4: footprint Connector_PinSocket_2.54mm:PinSocket_1x06_P2.54mm_Vertical -> Connector_PinHeader_2.54mm:PinHeader_1x06_P2.54mm_Vertical
- moved U3 84.8 mm to (92.7, 52.1), turned to 180 degrees
- moved R11 83.6 mm to (123.2, 46.0), turned to 180 degrees
- moved C7 82.9 mm to (120.7, 45.1), turned to -90 degrees
- moved D6 81.9 mm to (86.1, 41.5), turned to -45 degrees
- moved C6 78.7 mm to (93.1, 46.1), turned to 180 degrees
- moved R10 78.5 mm to (98.3, 49.3)
- moved R9 77.5 mm to (98.3, 47.8)
- moved Q3 74.8 mm to (90.0, 44.1), turned to 135 degrees
- moved U2 71.6 mm to (113.6, 56.7), turned to -90 degrees
- moved R7 71.4 mm to (121.7, 48.1)
- moved C8 69.8 mm to (117.2, 60.3), turned to -135 degrees
- moved R2 67.2 mm to (106.3, 59.3), turned to 180 degrees
- moved R6 65.5 mm to (122.0, 51.6), turned to 180 degrees
- moved D7 62.2 mm to (86.4, 87.2), turned to 45 degrees
- moved U1 60.5 mm to (106.0, 81.9), turned to 90 degrees
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Routing:
- net +BATT: track 0.00 -> 229.0 mm, vias 0 -> 5
- net GND: track 0.00 -> 218.5 mm, vias 0 -> 15
- net +3V3: track 0.00 -> 129.3 mm, vias 0 -> 6
- net VBUS: track 0.00 -> 85.1 mm, vias 0 -> 3
- net D-: track 0.00 -> 68.7 mm, vias 0 -> 5
- net D+: track 0.00 -> 66.6 mm, vias 0 -> 7
- net MOT_3: track 0.00 -> 58.9 mm, vias 0 -> 3
- net EN: track 0.00 -> 58.7 mm, vias 0 -> 3
- net SCL: track 0.00 -> 52.9 mm, vias 0 -> 1
- net MOT_2: track 0.00 -> 42.9 mm, vias 0 -> 3
- net SDA: track 0.00 -> 42.4 mm, vias 0 -> 5
- net MOT_1: track 0.00 -> 37.9 mm, vias 0 -> 1
- net MOT_4: track 0.00 -> 37.4 mm, vias 0 -> 3
- net SRV_2: track 0.00 -> 35.5 mm
- net RTS: track 0.00 -> 33.0 mm, vias 0 -> 2
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Other:
- board outline added: 99.8 x 99.8 mm
